Commit message: Limbs hsowing up in RViz, next step is integrating these limbs and their frames into the existing system

File: bimanual_controller/urdf/left_limb.xacro (robot description, xacro)
@@ -2,9 +2,9 @@
 <robot name="left_limb" xmlns:xacro="http://ros.org/wiki/xacro">
   <!-- Set your base link -->
-  <link name="base_link"/>
+  <link name="left_offset_link"/>
   <!-- Load Kinova Gen3 arm -->
   <xacro:include filename="$(find kortex_description)/arms/gen3/7dof/urdf/gen3_macro.xacro"/>
   <xacro:load_arm
-    parent="base_link"
+    parent="left_offset_link"
     dof="7"
     vision="false"

File: bimanual_controller/urdf/right_limb.xacro (robot description, xacro)
@@ -1,10 +1,26 @@
 <?xml version="1.0"?>
-<robot xmlns:xacro="http://ros.org/wiki/xacro" name="right_limb">
-  <xacro:include filename="$(find kinova_description)/urdf/kinova_gen3.urdf.xacro"/>
-  <xacro:include filename="$(find allegro_hand_description)/urdf/allegro_right.urdf.xacro"/>
-  <xacro:property name="prefix" value="right_" />
-  <!-- Kinova arm -->
-  <xacro:kinova_gen3 prefix="${prefix}" hand="none" />
-  <!-- Allegro hand -->
-  <xacro:allegro_right_hand parent="${prefix}end_effector_link" prefix="${prefix}" />
+<robot name="right_limb" xmlns:xacro="http://ros.org/wiki/xacro">
+  <!-- Set your base link -->
+  <link name="right_offset_link"/>
+  <!-- Load Kinova Gen3 arm -->
+  <xacro:include filename="$(find kortex_description)/arms/gen3/7dof/urdf/gen3_macro.xacro"/>
+  <xacro:load_arm
+    parent="right_offset_link"
+    dof="7"
+    vision="false"
+    prefix="right_"
+    robot_ip="0.0.0.0"
+    gripper_joint_name="right_gripper_joint"
+    use_fake_hardware="true">
+    <origin_xyz>0 0 0</origin_xyz>
+  </xacro:load_arm>
+  <!-- Load Allegro Hand (Right) -->
+  <xacro:include filename="$(find allegro_hand_description)/urdf/rightAllegroHand.urdf.xacro"/>
+  <xacro:right_allegro_hand
+    link_prefix="right_hand_"
+    joint_prefix="right_"
+    tip="default"
+    parent="right_end_effector_link">
+    <origin xyz="0 0 0.1" rpy="0 0 0"/>
+  </xacro:right_allegro_hand>
 </robot>
